File: Schematics/SmartButton.kicad_sch (KiCad schematic)
At the start: 33 parts, among them J1 Conn_01x02_Pin, J2 Conn_01x02_Pin, J3 Conn_01x02_Pin, Q1 2N2222, Q2 2N2222, Q3 2N2222, Q4 2N2222, SW1 SW_Push, U1 ESP32-WROOM-E, U2 XC6220B331MR

Commit message: Uograde to KiCad 9.0
Parts:
- U1: footprint PCM_Espressif:ESP32-WROOM-32E -> Espressif:ESP32-WROOM-32E
Changed lines of the file:
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@@
 (kicad_sch
-	(version 20231120)
+	(version 20250114)
 	(generator "eeschema")
-	(generator_version "8.0")
+	(generator_version "9.0")
 	(paper "A4")
 	(title_block
@@
 	(label "LED_ENABLE"
 		(at 261.62 40.64 180)
-		(fields_autoplaced yes)
 		(effects
 			(font
@@
 	(label "BOOT"
 		(at 261.62 35.56 180)
-		(fields_autoplaced yes)
 		(effects
 			(font
@@
 	(label "GND"
 		(at 212.09 83.82 90)
-		(fields_autoplaced yes)
 		(effects
 			(font
@@
 	(label "LED_DOUT"
 		(at 279.4 138.43 180)
-		(fields_autoplaced yes)
 		(effects
 			(font
@@
 	(label "SWITCH"
 		(at 261.62 55.88 180)
-		(fields_autoplaced yes)
 		(effects
 			(font
@@
 	(label "VBAT_MEASURE_ENABLE"
 		(at 17.78 86.36 0)
-		(fields_autoplaced yes)
 		(effects
 			(font
@@
 	(label "GND"
 		(at 39.37 36.83 180)
-		(fields_autoplaced yes)
 		(effects
 			(font
@@
 	(label "GND"
 		(at 74.93 190.5 180)
-		(fields_autoplaced yes)
 		(effects
 			(font
@@
 	(label "RX"
 		(at 261.62 30.48 180)
-		(fields_autoplaced yes)
 		(effects
 			(font
@@
 	(label "LED_DOUT"
 		(at 261.62 50.8 180)
-		(fields_autoplaced yes)
 		(effects
 			(font
@@
 	(label "VBAT_MEASURE_ADC1CH7"
 		(at 88.9 95.25 180)
-		(fields_autoplaced yes)
 		(effects
 			(font
@@
 	(label "VBAT+"
 		(at 52.07 33.02 0)
-		(fields_autoplaced yes)
 		(effects
 			(font
@@
 	(label "LED_DIN"
 		(at 144.78 138.43 0)
-		(fields_autoplaced yes)
 		(effects
 			(font
@@
 	(label "RTS"
 		(at 40.64 156.21 0)
-		(fields_autoplaced yes)
 		(effects
 			(font
@@
 	(label "LED_DIN"
 		(at 261.62 43.18 180)
-		(fields_autoplaced yes)
 		(effects
 			(font
@@
 	(label "33V"
 		(at 210.82 17.78 270)
-		(fields_autoplaced yes)
 		(effects
 			(font
@@
 	(label "GND"
 		(at 74.93 53.34 90)
-		(fields_autoplaced yes)
 		(effects
 			(font
@@
 	(label "GND"
 		(at 167.64 17.78 270)
-		(fields_autoplaced yes)
 		(effects
 			(font
@@
 	(label "VBAT+"
 		(at 60.96 62.23 270)
-		(fields_autoplaced yes)
 		(effects
 			(font
@@
 	(label "GND"
 		(at 30.48 40.64 270)
-		(fields_autoplaced yes)
 		(effects
 			(font
@@
 	(label "33V"
 		(at 78.74 116.84 270)
-		(fields_autoplaced yes)
 		(effects
 			(font
@@
 	(label "33V"
 		(at 49.53 172.72 270)
-		(fields_autoplaced yes)
 		(effects
 			(font
@@
 	(label "TX"
 		(at 261.62 27.94 180)
-		(fields_autoplaced yes)
 		(effects
 			(font
@@
 	(label "BOOT"
 		(at 90.17 167.64 180)
-		(fields_autoplaced yes)
 		(effects
 			(font
@@
 	(label "DTR"
 		(at 40.64 139.7 0)
-		(fields_autoplaced yes)
 		(effects
 			(font
@@
 	(label "VBAT_MEASURE_ENABLE"
 		(at 151.13 33.02 0)
-		(fields_autoplaced yes)
 		(effects
 			(font
@@
 	(label "SWITCH"
 		(at 151.13 48.26 0)
-		(fields_autoplaced yes)
 		(effects
 			(font
@@
 	(label "TX"
 		(at 269.24 30.48 0)
-		(fields_autoplaced yes)
 		(effects
 			(font
@@
 	(label "EN"
 		(at 151.13 27.94 0)
-		(fields_autoplaced yes)
 		(effects
 			(font
@@
 	(label "GND"
 		(at 60.96 111.76 90)
-		(fields_autoplaced yes)
 		(effects
 			(font
@@
 	(label "LED_ENABLE"
 		(at 182.88 101.6 0)
-		(fields_autoplaced yes)
 		(effects
 			(font
@@
 	(label "EN"
 		(at 90.17 130.81 180)
-		(fields_autoplaced yes)
 		(effects
 			(font
@@
 	(label "VBAT+"
 		(at 39.37 34.29 180)
-		(fields_autoplaced yes)
 		(effects
 			(font
@@
 	(label "33V"
 		(at 144.78 127 0)
-		(fields_autoplaced yes)
 		(effects
 			(font
@@
 	(label "GND"
 		(at 212.09 88.9 270)
-		(fields_autoplaced yes)
 		(effects
 			(font
@@
 	(label "LED_GND"
 		(at 212.09 107.95 270)
-		(fields_autoplaced yes)
 		(effects
 			(font
@@
 	(label "SWITCH"
 		(at 151.13 35.56 0)
-		(fields_autoplaced yes)
 		(effects
 			(font
@@
 	(label "VBAT_MEASURE_ADC1CH7"
 		(at 151.13 55.88 0)
-		(fields_autoplaced yes)
 		(effects
 			(font
@@
 	(label "33V"
 		(at 129.54 33.02 180)
-		(fields_autoplaced yes)
 		(effects
 			(font
@@
 	(label "LED_GND"
 		(at 212.09 161.29 90)
-		(fields_autoplaced yes)
 		(effects
 			(font
@@
 	(label "DTR"
 		(at 31.75 148.59 180)
-		(fields_autoplaced yes)
 		(effects
 			(font
@@
 	(label "RTS"
 		(at 31.75 146.05 180)
-		(fields_autoplaced yes)
 		(effects
 			(font
@@
 	(label "RX"
 		(at 269.24 27.94 0)
-		(fields_autoplaced yes)
 		(effects
 			(font
@@
 	(label "SWITCH"
 		(at 35.56 190.5 0)
-		(fields_autoplaced yes)
 		(effects
 			(font
@@
 	(label "GND"
 		(at 107.95 49.53 90)
-		(fields_autoplaced yes)
 		(effects
 			(font
@@
 			)
 		)
-		(property "Footprint" "PCM_Espressif:ESP32-WROOM-32E"
+		(property "Footprint" "Espressif:ESP32-WROOM-32E"
 			(at 210.82 83.82 0)
 			(effects
@@
 		)
 	)
+	(embedded_fonts no)
 )

Commit message: Label components in schematic as they appear on the board (R4 <-> R2, R7 <-> R5, R2 <-> R8) - Update PDF and SVG
Parts:
- renumbered R4 to R2, R8 to R4, R7 to R5, R5 to R7, R2 to R8
Changed lines of the file:
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@@
 	(title_block
 		(title "SmartButton")
-		(date "2024-07-20")
-		(rev "1")
+		(date "2025-08-24")
+		(rev "2")
 		(company "Gilles Zunino")
 		(comment 1 "Reversed Engineered from device")
@@
 		(on_board yes)
 		(dnp no)
-		(property "Reference" "R4"
+		(property "Reference" "R2"
 			(at 54.61 151.13 90)
 			(effects
@@
 			(project "SmartButton"
 				(path "/6b589a6a-2259-48e5-bd4a-c88d6ffe2aa8"
-					(reference "R4")
+					(reference "R2")
 					(unit 1)
 				)
@@
 		(dnp no)
 		(fields_autoplaced yes)
-		(property "Reference" "R7"
+		(property "Reference" "R5"
 			(at 63.5 72.3899 0)
 			(effects
@@
 			(project "SmartButton"
 				(path "/6b589a6a-2259-48e5-bd4a-c88d6ffe2aa8"
-					(reference "R7")
+					(reference "R5")
 					(unit 1)
 				)
@@
 		(dnp no)
 		(fields_autoplaced yes)
-		(property "Reference" "R2"
+		(property "Reference" "R8"
 			(at 81.28 123.1899 0)
 			(effects
@@
 			(project ""
 				(path "/6b589a6a-2259-48e5-bd4a-c88d6ffe2aa8"
-					(reference "R2")
+					(reference "R8")
 					(unit 1)
 				)
@@
 		(on_board yes)
 		(dnp no)
-		(property "Reference" "R8"
+		(property "Reference" "R4"
 			(at 46.99 80.518 90)
 			(effects
@@
 			(project "SmartButton"
 				(path "/6b589a6a-2259-48e5-bd4a-c88d6ffe2aa8"
-					(reference "R8")
+					(reference "R4")
 					(unit 1)
 				)
@@
 		(dnp no)
 		(fields_autoplaced yes)
-		(property "Reference" "R5"
+		(property "Reference" "R7"
 			(at 52.07 181.6099 0)
 			(effects
@@
 			(project "SmartButton"
 				(path "/6b589a6a-2259-48e5-bd4a-c88d6ffe2aa8"
-					(reference "R5")
+					(reference "R7")
 					(unit 1)
 				)

Commit message: Upgrade to KiCad 10
Parts:
- Q1, Q2, Q3, Q4: symbol Transistor_BJT_AKL:Q_NPN_Generic_BCE -> PCM_Transistor_BJT_AKL:Q_NPN_Generic_BCE
- U1: footprint Espressif:ESP32-WROOM-32E -> PCM_Espressif:ESP32-WROOM-32E; symbol Espressif:ESP32-WROOM-E -> PCM_Espressif:ESP32-WROOM-E
